Commit message: Added sensor to gripper model

File: models/george_gripper.urdf.xacro (robot description, xacro)
@@ -26,4 +26,5 @@
      <material>Gazebo/Orange</material>
    </gazebo>
+  <!-- Pads -->
    <link name="pad${suffix}">
     <visual>
@@ -87,7 +88,39 @@
       <material>Gazebo/Orange</material>
     </gazebo>
+       <!-- Contact sensor -->
+    <link name="contact_sensor_link">
+        <collision name="box_collision">
+            <origin xyz="0 0 0" rpy="0 0 0"/>
+            <geometry>
+                <box size = "0.02 0.04 0.26"/>
+            </geometry>
+        </collision>
+        <visual>
+            <origin xyz="0 0 0" rpy="0 0 0"/>
+            <geometry>
+                <box size = "0.02 0.04 0.26"/>
+            </geometry>
+        </visual>
+        <sensor name='my_contact' type='contact'>
+            <contact>
+                <collision>box_collision</collision>
+            </contact>
+            <always_on>1</always_on>
+            <update_rate>5</update_rate>
+            <!-- <visualize>true</visualize> !-->
+        </sensor>
+    </link>
+    <gazebo reference="contact_sensor_link">
+        <material>Gazebo/Red</material>
+    </gazebo>
     <!-- make two fingers -->
     <xacro:finger suffix="1" />
     <xacro:finger suffix="2" />
+    <!-- Join sensor to pad-->
+    <joint name="sensor1_to_pad1" type="fixed">
+      <parent link="pad1" />
+      <child link = "contact_sensor_link" />
+      <origin xyz="0.013 0 0.06" rpy="0 0 0"/>
+    </joint>
     <!-- fingers can slide -->
     <joint name="palm_to_finger1" type="prismatic">

Commit message: Correctly positioned sensor on gripper

File: models/george_gripper.urdf.xacro (robot description, xacro)
@@ -121,5 +121,5 @@
       <parent link="pad1" />
       <child link = "contact_sensor_link" />
-      <origin xyz="0.013 0 0.06" rpy="0 0 0"/>
+      <origin xyz="0.01 0 0.005" rpy="0 0 0"/>
     </joint>
     <!-- fingers can slide -->

Commit message: Contact sensor now pub to gazebo

File: models/george_gripper.urdf.xacro (robot description, xacro)
@@ -90,5 +90,5 @@
        <!-- Contact sensor -->
     <link name="contact_sensor_link">
-        <collision name="box_collision">
+        <collision name="contact_sensor_collision">
             <origin xyz="0 0 0" rpy="0 0 0"/>
             <geometry>
@@ -102,15 +102,15 @@
             </geometry>
         </visual>
-        <sensor name='my_contact' type='contact'>
-            <contact>
-                <collision>box_collision</collision>
-            </contact>
-            <always_on>1</always_on>
-            <update_rate>5</update_rate>
-            <!-- <visualize>true</visualize> !-->
-        </sensor>
     </link>
     <gazebo reference="contact_sensor_link">
-        <material>Gazebo/Red</material>
+        <sensor name='my_contact' type='contact'>
+          <always_on>1</always_on>
+          <update_rate>0.5</update_rate>
+          <contact>
+              <collision>contact_sensor_collision_collision</collision>
+              <topic>/contact_sensor</topic>
+          </contact>
+      </sensor>
+      <material>Gazebo/Red</material>
     </gazebo>
     <!-- make two fingers -->

Commit message: Reverted sensor addition

File: models/george_gripper.urdf.xacro (robot description, xacro)
@@ -88,5 +88,5 @@
       <material>Gazebo/Orange</material>
     </gazebo>
-       <!-- Contact sensor -->
+       <!-- Contact sensor
     <link name="contact_sensor_link">
         <collision name="contact_sensor_collision">
@@ -105,4 +105,5 @@
     <gazebo reference="contact_sensor_link">
         <sensor name='my_contact' type='contact'>
+          <plugin name="my_plugin" filename="libcontact.so"/>
           <always_on>1</always_on>
           <update_rate>0.5</update_rate>
@@ -113,14 +114,14 @@
       </sensor>
       <material>Gazebo/Red</material>
-    </gazebo>
+    </gazebo> -->
     <!-- make two fingers -->
     <xacro:finger suffix="1" />
     <xacro:finger suffix="2" />
-    <!-- Join sensor to pad-->
+    <!-- Join sensor to pad
     <joint name="sensor1_to_pad1" type="fixed">
       <parent link="pad1" />
       <child link = "contact_sensor_link" />
       <origin xyz="0.01 0 0.005" rpy="0 0 0"/>
-    </joint>
+    </joint> -->
     <!-- fingers can slide -->
     <joint name="palm_to_finger1" type="prismatic">
