Commit message: Updated camera_1 position

File: models/farscope_new_gripper_robot.urdf.xacro (robot description, xacro)
@@ -13,5 +13,5 @@
   <xacro:include filename="simple_camera.urdf.xacro" />
   <xacro:simple_camera camera_name="camera1" parent_link="forearm_link" >
-    <origin xyz="0 -0.08 0.38" rpy="0 -1.5706 0" />
+    <origin xyz="0 -0.08 0.565" rpy="0 -1.5706 0" />
   </xacro:simple_camera>
   <xacro:simple_camera camera_name="camera2" parent_link="upper_arm_link" >
